File: Board/ESP12E_EvalBoard.kicad_pcb (KiCad board)
At the start: 2 copper layers, 40 x 50 mm, 31 parts, among them J1 USB_OTG, J2 Conn_01x11, J3 Conn_01x11, SW1 SW_Reset, U1 ESP-12E, U2 NCP1117ST33T3G, U3 FT230XS

Commit message: Production version
Routing:
- net Net-(J2-Pad9): track 30.5 -> 29.7 mm
